Commit message: 0325cmd1_60000

File: dynamics/src/dynamics/urdf/single_arm_v22_19cm.urdf (robot description, URDF)
Before this commit: robot single_arm_v22_19cm, 8 links, 7 joints
Links:
- link link2: mass 1.33974234835036 -> 1.443911166204783
- link link3: mass 1.19767908022107 -> 1.3418327873616724
Joints:
- joint joint3: origin xyz=0.214867681425003 0 -0.039 rpy=0 0 0 -> xyz=0.29673382322145303 0 -0.039 rpy=0 0 0
- joint joint4: origin xyz=0.285132318574997 0 0.039 rpy=0 0 -3.14159265358979 -> xyz=0.39842253413401896 0 0.039 rpy=0 0 -3.14159265358979

File: dynamics/src/dynamics/urdf/single_arm_v22_19cm_motion.urdf (robot description, URDF)
Before this commit: robot single_arm_v22_19cm, 8 links, 7 joints
Links:
- link link2: mass 1.33974234835036 -> 1.443911166204783
- link link3: mass 1.19767908022107 -> 1.3418327873616724
Joints:
- joint joint3: origin xyz=0.214867681425003 0 -0.039 rpy=0 0 0 -> xyz=0.29673382322145303 0 -0.039 rpy=0 0 0
- joint joint4: origin xyz=0.285132318574997 0 0.039 rpy=0 0 -3.14159265358979 -> xyz=0.39842253413401896 0 0.039 rpy=0 0 -3.14159265358979
